Commit message: edited urdf file to get rid of errors, only issue now is shoulder joint being improperly defined

File: robot-sim/models_and_worlds/models/arm/arm.urdf (robot description, URDF)
Before this commit: robot arm, 6 links, 4 joints
Links:
- removed link elbow_linkage
Joints:
- joint shoulder_1: child shoulder_assembly -> bicep_actuator; parent bicep_actuator -> shoulder_assembly

Commit message: edited urdf file to get rid of errors, only issue now is shoulder joint being improperly defined

File: robot-sim/models_and_worlds/models/arm/arm.urdf (robot description, URDF)
Before this commit: robot arm, 6 links, 4 joints
Links:
- removed link elbow_linkage
- link bicep_actuator: geometry collision mesh filename=package://models_and_worlds/models/arm/assets/0_4m_shaft.stl; collision mesh filename=package://models_and_worlds/models/arm/assets/200mm_linear_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
- link forearm: geometry collision mesh filename=package://models_and_worlds/models/arm/assets/0_3m_shaft.stl; collision mesh filename=package://models_and_worlds/models/arm/assets/extrude_thin1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
- link gripper_assembly: geometry collision mesh filename=package://models_and_worlds/models/arm/assets/1911_0025_083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; collision mesh filename=package://models_and_worlds/models/arm/assets/1911_0025_083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
- link joint: geometry collision mesh filename=package://models_and_worlds/models/arm/assets/deleteface2.s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; collision mesh filename=package://models_and_worlds/models/arm/assets/part_1__26.stl
- link shoulder_assembly: geometry collision mesh filename=package://models_and_worlds/models/arm/assets/1mt_054_006.s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; collision mesh filename=package://models_and_worlds/models/arm/assets/1mt_054_006__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
Joints:
- joint shoulder_1: child shoulder_assembly -> bicep_actuator; parent bicep_actuator -> shoulder_assembly

Commit message: Fixed arm asset paths

File: robot-sim/models_and_worlds/models/arm/arm.urdf (robot description, URDF)
Before this commit: robot arm, 5 links, 4 joints
Links:
- link bicep_actuator: geometry collision mesh filename=package://models_and_worlds/models/arm/assets/0_4m_shaft.stl; collision mesh filename=package://models_and_worlds/models/arm/assets/200mm_linear_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
- link forearm: geometry collision mesh filename=package://models_and_worlds/models/arm/assets/0_3m_shaft.stl; collision mesh filename=package://models_and_worlds/models/arm/assets/extrude_thin1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
- link gripper_assembly: geometry collision mesh filename=package://models_and_worlds/models/arm/assets/1911_0025_083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; collision mesh filename=package://models_and_worlds/models/arm/assets/1911_0025_083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
- link joint: geometry collision mesh filename=package://models_and_worlds/models/arm/assets/deleteface2.s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; collision mesh filename=package://models_and_worlds/models/arm/assets/part_1__26.stl
- link shoulder_assembly: geometry collision mesh filename=package://models_and_worlds/models/arm/assets/1mt_054_006.s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; collision mesh filename=package://models_and_worlds/models/arm/assets/1mt_054_006__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

Commit message: Added base link joint to arm urdf file

File: robot-sim/models_and_worlds/models/arm/arm.urdf (robot description, URDF)
Before this commit: robot arm, 5 links, 4 joints
Links:
- added link base_link
Joints:
- added joint base_to_shoulder: type fixed, parent base_link, child shoulder_assembly, origin xyz=0 0 0 rpy=0 0 0
