Commit message: Added joint controller 🥳

File: robot-sim/models_and_worlds/models/arm/preview.urdf (robot description, URDF)
Before this commit: robot arm, 6 links, 5 joints
Links:
- removed link base_link
- link bicep_actuator: geometry collision mesh filename=assets/0_4m_shaft.stl; collision mesh filename=assets/200mm_linear_actuator_base.stl
- link forearm: geometry collision mesh filename=assets/0_3m_shaft.stl; collision mesh filename=assets/extrude_thin1.stl
- link gripper_assembly: geometry collision mesh filename=assets/1911_0025_0836_assembly.stl; collision mesh filename=assets/1911_0025_0836_assembly__2.stl
- link joint: geometry collision mesh filename=assets/deleteface2.stl; collision mesh filename=assets/part_1__26.stl
- link shoulder_assembly: geometry collision mesh filename=assets/1mt_054_006.stl; collision mesh filename=assets/1mt_054_006__2.stl
Joints:
- removed joint base_to_shoulder
