Commit message: RESTRUCTURE

File: robot-sim/arm_description/urdf/arm.urdf (robot description, URDF)
Before this commit: robot arm, 5 links, 4 joints
Links:
- added link base_link
- link bicep_actuator: geometry collision mesh filename=${mesh_path}/0_4m_shaft.stl; collision mesh filename=${mesh_path}/200mm_linear_actuator_base.stl
- link forearm: geometry collision mesh filename=${mesh_path}/0_3m_shaft.stl; collision mesh filename=${mesh_path}/extrude_thin1.stl
- link gripper_assembly: geometry collision mesh filename=${mesh_path}/1911_0025_0836_assembly.stl; collision mesh filename=${mesh_path}/1911_0025_0836_assembly__2.stl
- link joint: geometry collision mesh filename=${mesh_path}/deleteface2.stl; collision mesh filename=${mesh_path}/part_1__26.stl
- link shoulder_assembly: geometry collision mesh filename=${mesh_path}/1mt_054_006.stl; collision mesh filename=${mesh_path}/1mt_054_006__2.stl
Joints:
- added joint base_to_shoulder: type fixed, parent base_link, child shoulder_assembly, origin xyz=0 0 0 rpy=0 0 0

Commit message: Made genbot work, rebuild arm packages using gebot

File: robot-sim/arm_description/urdf/arm.urdf (robot description, URDF)
Before this commit: robot arm, 6 links, 5 joints
Links:
- added link elbow_linkage, mass 0.0164299; collision mesh filename=${mesh_path}/actuator_linkage.stl; collision mesh filename=${mesh_path}/actuator_linkage.stl
- link base_link: mass None -> 1e-09
- link bicep_actuator: geometry collision mesh filename=${mesh_path}/0_4m_shaft.stl; collision mesh filename=${mesh_path}/200mm_linear_actuator_base.stl
- link shoulder_assembly: mass 2.79424 -> 2.78799; geometry collision mesh filename=${mesh_path}/1mt_054_006.stl; collision mesh filename=${mesh_path}/1mt_054_006__2.stl
Joints:
- removed joint base_to_shoulder
- added joint base_link_to_elbow_linkage: type fixed, parent base_link, child elbow_linkage, origin xyz=0 0 0 rpy=0 -0 0, axis 0 0 1, limit effort=10 velocity=10
- added joint base_link_to_shoulder_assembly: type fixed, parent base_link, child shoulder_assembly, origin xyz=0 0 0 rpy=0 -0 0, axis 0 0 1, limit effort=10 velocity=10
- joint elbow_1: origin xyz=-0.0075 -0.379629 0.135874 rpy=-1.5708 0.111404 1.5708 -> xyz=0.219114 -0.313521 -0.018175 rpy=-0 -0 2.18077
- joint shoulder_1: origin xyz=-0.025675 0.000500014 0.09335 rpy=-1.5708 2.77556e-16 -1.5708 -> xyz=-0.025675 0.000500014 0.09335 rpy=1.5708 -1.179 -1.5708
- joint wrist_1: origin xyz=-0.278802 0.209514 0.0265 rpy=6.15077e-16 1.98812e-14 2.49714 -> xyz=-0.317969 -0.143256 0.0265 rpy=-0 0 -2.7183
- joint wrist_2: origin xyz=0.00664496 0.00408467 -0.034 rpy=-1.5708 1.16626 -1.01964 -> xyz=-0.00623455 -0.00468726 -0.034 rpy=-1.5708 1.16626 2.21546

File: robot-sim/arm_description/urdf/arm_control.urdf.xacro (robot description, xacro)
@@ -6,5 +6,16 @@
             <plugin>gz_ros2_control/GazeboSimSystem</plugin>
         </hardware>
-        <joint name="shoulder_1">
+        <joint name="wrist_2">
+            <command_interface name="position">
+                <param name="min">-3.14</param>
+                <param name="max">3.14</param>
+            </command_interface>
+            <state_interface name="position">
+                <param name="initial_value">1.0</param>
+            </state_interface>
+            <state_interface name="velocity"/>
+            <state_interface name="effort"/>
+        </joint>
+        <joint name="wrist_1">
             <command_interface name="position">
                 <param name="min">-3.14</param>
@@ -28,16 +39,5 @@
             <state_interface name="effort"/>
         </joint>
-        <joint name="wrist_1">
-            <command_interface name="position">
-                <param name="min">-3.14</param>
-                <param name="max">3.14</param>
-            </command_interface>
-            <state_interface name="position">
-                <param name="initial_value">1.0</param>
-            </state_interface>
-            <state_interface name="velocity"/>
-            <state_interface name="effort"/>
-        </joint>
-        <joint name="wrist_2">
+        <joint name="shoulder_1">
             <command_interface name="position">
                 <param name="min">-3.14</param>
