Commit message: Save all changes

File: robot-sim/arm_description/urdf/arm_control.urdf.xacro (robot description, xacro)
@@ -1,4 +1,7 @@
 <?xml version="1.0" ?>
 <robot xmlns:xacro="http://www.ros.org/wiki/xacro" name="arm_control">
+    <xacro:arg name="controller_config" default=""/>
+    <xacro:arg name="plugin_extension" default=".so"/>
+    <xacro:property name="plugin_extension" value="$(arg plugin_extension)"/>
     <!-- ros2_control hardware interface -->
     <ros2_control name="GazeboSimSystem" type="system">
@@ -53,5 +56,5 @@
     <gazebo>
         <!-- JOINT CONTROLLER -->
-        <plugin filename="libgz_ros2_control-system.so" name="gz_ros2_control::GazeboSimROS2ControlPlugin">
+        <plugin filename="libgz_ros2_control-system${plugin_extension}" name="gz_ros2_control::GazeboSimROS2ControlPlugin">
             <robot_param>robot_description</robot_param>
             <robot_param_node>robot_state_publisher</robot_param_node>
