Commit message: updating generation of model to properly reference meshes for genesis

File: robot-sim/arm/urdf/arm.urdf (robot description, URDF)
Before this commit: robot arm, 8 links, 7 joints
Links:
- link bicep_actuator: geometry collision mesh filename=../meshes/0_4m_shaft.stl; collision mesh filename=../meshes/200mm_linear_actuator_base.stl
- link elbow_linkage: geometry collision mesh filename=../meshes/actuator_linkage.stl; collision mesh filename=../meshes/actuator_linkage.stl
- link forearm: geometry collision mesh filename=../meshes/0_3m_shaft.stl; collision mesh filename=../meshes/extrude_thin1.stl
- link gripper_assembly: geometry collision mesh filename=../meshes/1911_0025_0836_assembly.stl; collision mesh filename=../meshes/1911_0025_0836_assembly__2.stl
- link joint: geometry collision mesh filename=../meshes/deleteface2.stl; collision mesh filename=../meshes/part_1__26.stl
- link shoulder_assembly: geometry collision mesh filename=../meshes/1mt_054_006.stl; collision mesh filename=../meshes/1mt_054_006__2.stl

Commit message: Fixed some mesh reference issues and made joint updates smooth instead of teleport

File: robot-sim/arm/urdf/arm.urdf (robot description, URDF)
Before this commit: robot arm, 8 links, 7 joints
Links:
- link bicep_actuator: geometry collision mesh filename=package://arm/meshes/0_4m_shaft.stl; collision mesh filename=package://arm/meshes/200mm_linear_actuator_base.stl
- link elbow_linkage: geometry collision mesh filename=package://arm/meshes/actuator_linkage.stl; collision mesh filename=package://arm/meshes/actuator_linkage.stl
- link forearm: geometry collision mesh filename=package://arm/meshes/0_3m_shaft.stl; collision mesh filename=package://arm/meshes/extrude_thin1.stl
- link gripper_assembly: geometry collision mesh filename=package://arm/meshes/1911_0025_0836_assembly.stl; collision mesh filename=package://arm/meshes/1911_0025_0836_assembly__2.stl
- link joint: geometry collision mesh filename=package://arm/meshes/deleteface2.stl; collision mesh filename=package://arm/meshes/part_1__26.stl
- link shoulder_assembly: geometry collision mesh filename=package://arm/meshes/1mt_054_006.stl; collision mesh filename=package://arm/meshes/1mt_054_006__2.stl

Commit message: resolved merge

File: robot-sim/arm/urdf/arm.urdf (robot description, URDF)
Before this commit: robot arm, 8 links, 7 joints
Joints:
- removed joint base_link_to_elbow_linkage
- added joint bicep_to_elbow_linkage: type continuous, parent bicep_actuator, child elbow_linkage, origin xyz=-0.08608547 -0.03610776 -0.02567487 rpy=2.945694 1.570795 -2.945694, axis 0 0 1, limit effort=10 velocity=10
